File: PCBDesign/AirLoRaV3_PCBDesign/_autosave-Power.kicad_sch (KiCad schematic)
At the start: 16 parts, among them J1 Barrel_Jack_Switch_Pin3Ring, U1 TPS7A2633DRVR, U4 TPS54202DDC

Commit message: Updated Schematic
Parts:
- added C3: 75pF, Capacitor_Tantalum_SMD:CP_EIA-6032-15_Kemet-U, symbol Device:C_Small
- added C5: 22uF, Capacitor_Tantalum_SMD:CP_EIA-6032-15_Kemet-U, symbol Device:C_Small
- added R1: 100K, symbol Device:R
- C1: value 470uF -> 10uF
- C2: renamed from C14; value 470uF -> 0.1uF
- C4: renamed from C15; value 100Uf -> 0.1uF
- C6: renamed from C2; value 100Uf -> 22uF
- L1: value 68uH -> 15uH
- R2: renamed from R7; value R -> 13.3K
- R3: renamed from R6; value R -> 49.9
- R4: renamed from R10; value R -> 10K
- R5: renamed from R8; value R -> 1.96M
- R6: renamed from R9; value R -> 1.18M
- renumbered C3 to C7, C5 to C8, U4 to U1, U1 to U2
Connections:
- net 5V: now also R3.2, C5.1
- net GND: now also U2.7 (EXP), C5.2
- net at C4.2, L1.1, U1.2 (SW): no longer R3.1
- net at R2.1, U1.4 (FB): now also C3.2, R1.2; no longer R3.2
- new net: C3.1, R1.1, R3.1
Other:
- moved on the sheet: C1, C2, C4, C6, C7, C8, D1, J1, L1, R2, R3, R4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
