File: PCBDesign/AirLoRaV3_PCBDesign/airlora-kicad.kicad_pcb (KiCad board)
At the start: 2 copper layers, 0 parts

Commit message: Update PCB layout
Parts:
- added C1: 10uF, Capacitor_SMD:C_1206_3216Metric_Pad1.33x1.80mm_HandSolder, F.Cu at (68.6, 92.8)
- added C10: 3.3pF, Capacitor_SMD:C_0603_1608Metric, F.Cu at (111.6, 92.2)
- added C11: 33pF, Capacitor_SMD:C_0603_1608Metric, F.Cu at (109.0, 91.5)
- added C12: 1nF, Capacitor_SMD:C_0603_1608Metric, F.Cu at (106.3, 93.9)
- added C13: 10pF, Capacitor_SMD:C_0603_1608Metric, F.Cu at (107.3, 86.9)
- added C14: 10pF, Capacitor_SMD:C_0603_1608Metric, F.Cu at (106.3, 95.5)
- added C15: 1nF, Capacitor_SMD:C_0603_1608Metric, F.Cu at (107.3, 88.4)
- added C16: 12.5pF, Capacitor_SMD:C_0603_1608Metric, F.Cu at (92.5, 90.2)
- added C17: 68pF, Capacitor_SMD:C_0603_1608Metric, F.Cu at (101.8, 83.8)
- added C18: 100nF, Capacitor_SMD:C_0603_1608Metric, F.Cu at (87.6, 73.2)
- added C19: 470nF, Capacitor_SMD:C_0603_1608Metric, F.Cu at (90.5, 81.0)
- added C2: 0.1uF, Capacitor_SMD:C_0603_1608Metric, F.Cu at (70.6, 92.2)
- added C20: 4.7uF, Capacitor_SMD:C_0603_1608Metric, F.Cu at (95.9, 76.8)
- added C21: 100pF, Capacitor_SMD:C_0603_1608Metric, F.Cu at (101.8, 88.4)
- added C22: 12.5pF, Capacitor_SMD:C_0603_1608Metric, F.Cu at (94.7, 90.2)
- added C23: 47pF, Capacitor_SMD:C_0603_1608Metric, F.Cu at (101.8, 85.3)
- added C24: 100nF, Capacitor_SMD:C_0603_1608Metric, F.Cu at (99.0, 76.8)
- added C25: 100nF, Capacitor_SMD:C_0603_1608Metric, F.Cu at (92.9, 76.8)
- added C26: 100nF, Capacitor_SMD:C_0603_1608Metric, F.Cu at (101.8, 76.2)
- added C27: 100nF, Capacitor_SMD:C_0603_1608Metric, F.Cu at (94.4, 76.8)
- added C28: 4.7uF, Capacitor_SMD:C_0603_1608Metric, F.Cu at (101.8, 79.2)
- added C29: 100nF, Capacitor_SMD:C_0603_1608Metric, F.Cu at (97.5, 76.8)
- added C3: 75pF, Capacitor_SMD:C_0603_1608Metric, F.Cu at (78.9, 94.3)
- added C30: 100nF, Capacitor_SMD:C_0603_1608Metric, F.Cu at (101.8, 80.8)
- added C31: 10pF, Capacitor_SMD:C_0603_1608Metric, F.Cu at (89.6, 91.7)
- added C32: 5.1pF, Capacitor_SMD:C_0603_1608Metric, F.Cu at (86.2, 88.7)
- added C33: 10pF, Capacitor_SMD:C_0603_1608Metric, F.Cu at (89.6, 93.2)
- added C34: 10pF, Capacitor_SMD:C_0603_1608Metric, F.Cu at (86.2, 85.7)
- added C35: 4.7uF, Capacitor_SMD:C_0603_1608Metric, F.Cu at (91.4, 76.8)
- added C36: 100nF, Capacitor_SMD:C_0603_1608Metric, F.Cu at (101.8, 82.3)
- added C37: 33pF, Capacitor_SMD:C_0603_1608Metric, F.Cu at (96.3, 88.0)
- added C38: 33pF, Capacitor_SMD:C_0603_1608Metric, F.Cu at (90.5, 84.1)
- added C39: 100nF, Capacitor_SMD:C_0603_1608Metric, F.Cu at (90.5, 82.6)
- added C4: 0.1uF, Capacitor_SMD:C_0603_1608Metric, F.Cu at (76.4, 93.5)
- added C40: 33pF, Capacitor_SMD:C_0603_1608Metric, F.Cu at (97.9, 88.0)
- added C5: 22uF, Capacitor_SMD:C_1206_3216Metric_Pad1.33x1.80mm_HandSolder, F.Cu at (72.6, 82.4)
- added C6: 22uF, Capacitor_SMD:C_0603_1608Metric, F.Cu at (72.5, 80.3)
- added C7: 1uF, Capacitor_SMD:C_1206_3216Metric_Pad1.33x1.80mm_HandSolder, F.Cu at (77.4, 77.2)
- added C8: 1uF, Capacitor_SMD:C_1206_3216Metric_Pad1.33x1.80mm_HandSolder, F.Cu at (80.0, 72.0)
- added C9: 3.3pF, Capacitor_SMD:C_0603_1608Metric, F.Cu at (116.9, 92.2)
- added D1: 1N4007, Diode_SMD:D_SMA, F.Cu at (70.2, 101.3)
- added D2: LED, LED_SMD:LED_0603_1608Metric_Pad1.05x0.95mm_HandSolder, F.Cu at (70.5, 73.3)
- added D3: LED, LED_SMD:LED_0603_1608Metric_Pad1.05x0.95mm_HandSolder, F.Cu at (70.5, 67.8)
- added H1: MountingHole_Pad, MountingHole:MountingHole_3mm_Pad_Via, F.Cu at (119.0, 108.0)
- added H2: MountingHole_Pad, MountingHole:MountingHole_3mm_Pad_Via, F.Cu at (119.0, 58.0)
- added H3: MountingHole_Pad, MountingHole:MountingHole_3mm_Pad_Via, F.Cu at (69.0, 108.0)
- added H4: MountingHole_Pad, MountingHole:MountingHole_3mm_Pad_Via, F.Cu at (69.0, 58.0)
- added IC1: BALFHB-WL-05D3, footprint:BALFHBWL05D3, F.Cu at (102.8, 91.5)
- added J1: 12V, Connector_Phoenix_MC:PhoenixContact_MCV_1,5_2-G-3.5_1x02_P3.50mm_Vertical, F.Cu at (77.6, 106.3)
- added J2: Conn_Coaxial, Connector_Coaxial:U.FL_Molex_MCRF_73412-0110_Vertical, F.Cu at (120.5, 91.5)
- added J3: DHT, Connector_JST:JST_XH_B3B-XH-A_1x03_P2.50mm_Vertical, F.Cu at (105.5, 60.5)
- added J4: UART1, Connector_JST:JST_XH_B4B-XH-A_1x04_P2.50mm_Vertical, F.Cu at (91.8, 60.5)
- added J5: UART2, Connector_JST:JST_XH_B4B-XH-A_1x04_P2.50mm_Vertical, F.Cu at (89.2, 105.0)
- added J6: I2C, Connector_JST:JST_XH_B4B-XH-A_1x04_P2.50mm_Vertical, F.Cu at (104.0, 105.0)
- added J7: UART2, Connector_JST:JST_XH_B4B-XH-A_1x04_P2.50mm_Vertical, F.Cu at (77.9, 60.5)
- added L1: 15uH, Inductor_SMD:L_Vishay_IHLP-2020, F.Cu at (72.6, 87.0)
- added L2: 8.7uH, Inductor_SMD:L_0603_1608Metric, F.Cu at (114.3, 91.5)
- added L3: 15uH, Capacitor_SMD:C_0603_1608Metric_Pad1.08x0.95mm_HandSolder, F.Cu at (90.5, 79.5)
- added L4: 600R@100MHz, Inductor_SMD:L_0603_1608Metric, F.Cu at (101.8, 77.7)
- added L5: 1400R 1GHz, Inductor_SMD:L_0603_1608Metric, F.Cu at (89.6, 90.2)
- added Q1: S8050, Package_TO_SOT_SMD:SOT-23, F.Cu at (113.0, 67.1)
- added Q2: S8050, Package_TO_SOT_SMD:SOT-23, F.Cu at (101.2, 67.1)
- added Q3: S8050, Package_TO_SOT_SMD:SOT-23, F.Cu at (89.5, 99.9)
- added Q4: S8050, Package_TO_SOT_SMD:SOT-23, F.Cu at (104.2, 99.9)
- added R1: 1k, Resistor_SMD:R_0603_1608Metric, F.Cu at (73.7, 96.3)
- added R10: 100, Resistor_SMD:R_0603_1608Metric, F.Cu at (106.3, 97.0)
- added R11: 100, Resistor_SMD:R_0603_1608Metric, F.Cu at (101.8, 86.9)
- added R12: 220, Resistor_SMD:R_0603_1608Metric, F.Cu at (86.2, 87.2)
- added R14: 1K, Resistor_SMD:R_0603_1608Metric, F.Cu at (113.3, 69.8)
- added R15: 1K, Resistor_SMD:R_0603_1608Metric, F.Cu at (101.5, 69.9)
- added R16: 1K, Resistor_SMD:R_0603_1608Metric, F.Cu at (86.1, 98.7)
- added R17: 1K, Resistor_SMD:R_0603_1608Metric, F.Cu at (100.9, 98.7)
- added R2: 100K, Resistor_SMD:R_0603_1608Metric, F.Cu at (78.9, 92.8)
- added R3: 13.3K, Resistor_SMD:R_0603_1608Metric, F.Cu at (79.6, 90.4)
- added R4: 49.9, Resistor_SMD:R_0603_1608Metric, F.Cu at (78.0, 90.4)
- added R5: 1k, Resistor_SMD:R_0603_1608Metric, F.Cu at (70.3, 74.9)
- added R6: 10K, Resistor_SMD:R_0603_1608Metric, F.Cu at (76.0, 71.0)
- added R7: 1.96M, Resistor_SMD:R_0603_1608Metric, F.Cu at (76.0, 69.4)
- added R8: 1.18M, Resistor_SMD:R_0603_1608Metric, F.Cu at (76.0, 67.9)
- added R9: 1k, Resistor_SMD:R_0603_1608Metric, F.Cu at (70.4, 69.4)
- added SW1: SW_Push, Button_Switch_SMD:SW_Push_1P1T_NO_Vertical_Wuerth_434133025816, F.Cu at (87.2, 70.2)
- added U1: TPS54202DDC, Package_TO_SOT_SMD:SOT-23-6, F.Cu at (73.6, 92.2)
- added U2: TPS7A2633DRVR, footprint:TPS7A2633DRVR, F.Cu at (76.0, 74.0)
- added U3: BGS12WN6E6327, footprint:BGS12SN6E6327XTSA1, F.Cu at (105.9, 91.5)
- added U4: STM32WLE5JCIx, Package_BGA:ST_UFBGA-73_5x5mm_Layout9x9_P0.5mm, F.Cu at (96.0, 82.5)
- added XTAL1: NT2016SA-32M-END4263A, footprint:NT2016SA-32M-END4263A_NDK, F.Cu at (89.5, 87.5)
- added Y1: NX2012SA 32.768KHz, footprint:XTAL_NX2012SA-32.768K-STD-MUB-1, F.Cu at (93.7, 87.7)
Routing:
- net +5V: track 0.00 -> 133.2 mm, vias 0 -> 4
- net VDDRF: track 0.00 -> 78.5 mm, vias 0 -> 13
- net /AirLora V3/MCU/PB9_SDA: track 0.00 -> 37.8 mm, vias 0 -> 1
- net /AirLora V3/MCU/PA12: track 0.00 -> 37.8 mm, vias 0 -> 2
- net 12V: track 0.00 -> 36.5 mm
- net /AirLora V3/MCU/PA9_TX: track 0.00 -> 32.7 mm, vias 0 -> 1
- net /AirLora V3/MCU/PB8_SCL: track 0.00 -> 31.4 mm, vias 0 -> 1
- net Net-(U4-NRST): track 0.00 -> 28.2 mm, vias 0 -> 2
- net /AirLora V3/MCU/T_SWDIO: track 0.00 -> 27.4 mm, vias 0 -> 1
- net /AirLora V3/MCU/T_SWCLK: track 0.00 -> 27.2 mm, vias 0 -> 1
- net /AirLora V3/MCU/PA11: track 0.00 -> 25.1 mm, vias 0 -> 1
- net /AirLora V3/MCU/PA5: track 0.00 -> 25.1 mm, vias 0 -> 2
- net /AirLora V3/MCU/PB2: track 0.00 -> 24.7 mm, vias 0 -> 3
- net /AirLora V3/MCU/PA10_RX: track 0.00 -> 24.2 mm, vias 0 -> 1
- net /AirLora V3/MCU/PA2_TX: track 0.00 -> 23.2 mm, vias 0 -> 1
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- added copper zone on F.Cu, net +5V
- added copper zone on F.Cu, net 12V
- added copper zone on B.Cu, net GND
- added copper zone on F.Cu, net GND
- added copper zone on In1.Cu, net GND
- added copper zone on In2.Cu, net GND
- added copper zone on F.Cu, net SW
- added copper zone on In2.Cu, net VDDPA
- added copper zone on F.Cu, net VDDRF
Other:
- board outline added: 60 x 60 mm
- copper layers 2 -> 4
