File: PCBDesign/AirLoRaV3_PCBDesign/_autosave-airlora-kicad.kicad_pcb (KiCad board)
At the start: 4 copper layers, 60 x 60 mm, 89 parts, among them IC1 BALFHB-WL-05D3, J1 12V, J2 Conn_Coaxial, J3 DHT, J4 UART1, J5 UART2, J6 I2C, J7 UART2, Q1 S8050, Q2 S8050, Q3 S8050, Q4 S8050, SW1 SW_Push, U1 TPS54202DDC, U2 TPS7A2633DRVR, U3 BGS12WN6E6327, U4 STM32WLE5JCIx, Y1 NX2012SA 32.768KHz

Commit message: Update schematic
Parts:
- added REF**: SW_E-Switch_EG1271_SPDT, Button_Switch_THT:SW_E-Switch_EG1271_SPDT, F.Cu at (174.4, 82.1)

Commit message: Update circuit buck converter and sensor
Parts:
- removed the C17 at (162.3, 88.8)
- removed the C23 at (162.3, 90.3)
- removed the C31 at (150.1, 96.7)
- removed the C33 at (150.1, 98.2)
- removed the C35 at (151.9, 81.7)
- removed the C36 at (162.3, 87.3)
- removed L5: 1400R 1GHz, Inductor_SMD:L_0603_1608Metric
- removed REF**: SW_E-Switch_EG1271_SPDT, Button_Switch_THT:SW_E-Switch_EG1271_SPDT
- removed the U4 at (156.5, 87.5)
- removed XTAL1: NT2016SA-32M-END4263A, footprint:NT2016SA-32M-END4263A_NDK
- added C2: 1uF, Capacitor_SMD:C_0805_2012Metric_Pad1.18x1.45mm_HandSolder, F.Cu at (84.5, 69.5)
- added C20: 0.47uF, Capacitor_SMD:C_0603_1608Metric, F.Cu at (68.8, 133.7)
- added C30: 100nF, Capacitor_SMD:C_0603_1608Metric, F.Cu at (68.8, 135.2)
- added C40: 100nf, Capacitor_SMD:C_0603_1608Metric, F.Cu at (241.3, 51.6)
- added C41: 100nf, Capacitor_SMD:C_0603_1608Metric, F.Cu at (235.4, 55.4)
- added C42: 100nf, Capacitor_SMD:C_0603_1608Metric, F.Cu at (252.9, 56.5)
- added C43: 100nf, Capacitor_SMD:C_0603_1608Metric, F.Cu at (246.8, 67.3)
- added C44: 100nf, Capacitor_SMD:C_0603_1608Metric, F.Cu at (235.2, 61.5)
- added C45: 22PF, Capacitor_SMD:C_0603_1608Metric, F.Cu at (228.1, 61.6)
- added C46: 22PF, Capacitor_SMD:C_0603_1608Metric, F.Cu at (228.1, 55.7)
- added C47: 100nF, Capacitor_SMD:C_0603_1608Metric, F.Cu at (215.2, 56.2)
- added C7: 1uF, Capacitor_SMD:C_0805_2012Metric_Pad1.18x1.45mm_HandSolder, F.Cu at (84.3, 64.0)
- added D3: LED, LED_SMD:LED_0603_1608Metric_Pad1.05x0.95mm_HandSolder, F.Cu at (68.5, 79.4)
- added D5: LED, LED_SMD:LED_0603_1608Metric_Pad1.05x0.95mm_HandSolder, F.Cu at (222.6, 58.3)
- added J3: Led, Connector_Molex:Molex_CLIK-Mate_502585-0370_1x03-1MP_P1.50mm_Horizontal, F.Cu at (49.1, 28.9)
- added J6: I2C, Connector_Molex:Molex_CLIK-Mate_502585-0470_1x04-1MP_P1.50mm_Horizontal, F.Cu at (34.3, 28.9)
- added Q1: ZVP2106GTA, Package_TO_SOT_SMD:SOT-223-3_TabPin2, F.Cu at (89.4, 96.6)
- added Q2: S8050, Package_TO_SOT_SMD:SOT-23, F.Cu at (42.7, 124.4)
- added Q3: S8050, Package_TO_SOT_SMD:SOT-23, F.Cu at (45.5, 37.6)
- added Q6: S8050, Package_TO_SOT_SMD:SOT-23, F.Cu at (30.0, 37.6)
- added R1: 10K, Resistor_SMD:R_0603_1608Metric, F.Cu at (82.5, 99.1)
- added R10: 1k, Resistor_SMD:R_0603_1608Metric, F.Cu at (68.5, 81.0)
- added R18: 1K, Resistor_SMD:R_0603_1608Metric, F.Cu at (204.3, 106.3)
- added R19: 1K, Resistor_SMD:R_0603_1608Metric, F.Cu at (39.1, 123.5)
- added R20: 1K, Resistor_SMD:R_0603_1608Metric, F.Cu at (50.0, 36.4)
- added R24: 1K, Resistor_SMD:R_0603_1608Metric, F.Cu at (34.4, 36.4)
- added R27: 1k, Resistor_SMD:R_0603_1608Metric, F.Cu at (222.6, 59.9)
- added R28: 10k, Resistor_SMD:R_0603_1608Metric, F.Cu at (215.2, 61.4)
- added R29: 10k, Resistor_SMD:R_0603_1608Metric, F.Cu at (221.9, 63.8)
- added R5: 10K, Resistor_SMD:R_0603_1608Metric, F.Cu at (77.0, 66.4)
- added R7: 1.96M, Resistor_SMD:R_0603_1608Metric, F.Cu at (80.0, 66.4)
- added R8: 1.18M, Resistor_SMD:R_0603_1608Metric, F.Cu at (80.1, 68.1)
- added SW2: SW_Slide_DPDT, Button_Switch_THT:SW_E-Switch_EG1271_SPDT, F.Cu at (104.5, 67.9)
- added SW3: SW_Push, Button_Switch_SMD:SW_Push_SPST_NO_Alps_SKRK, F.Cu at (214.0, 58.8)
- added U2: TPS7A2633DRVR, footprint:TPS7A2633DRVR, F.Cu at (84.3, 66.7)
- added U5: STM32WLE5CCUx, Package_DFN_QFN:QFN-48-1EP_7x7mm_P0.5mm_EP5.6x5.6mm, F.Cu at (77.3, 137.5)
- added U6: STM32F103C8Tx, Package_QFP:LQFP-48_7x7mm_P0.5mm, F.Cu at (244.1, 59.3)
- added X1: NX2016SA-32MHZ, footprint:NX2016SA_NDK, F.Cu at (86.8, 142.5)
- added Y2: 8Mhz, Crystal:Crystal_SMD_3225-4Pin_3.2x2.5mm, F.Cu at (228.2, 58.6)
- C18: renamed from C32; value 5.1pF -> 6.8pF
- C24: renamed from C34; value 10pF -> 6.8pF
- C29: value 100nF -> 4.7uF
- C39: value 100nF -> 4.7uf; footprint Capacitor_SMD:C_0603_1608Metric -> Capacitor_SMD:C_0805_2012Metric
- D1: value 1N4007 -> D_Zener; footprint Diode_SMD:D_SMA -> Diode_SMD:D_SMA_Handsoldering
- IC1: value BALFHB-WL-05D3 -> BALFHB-WL-02D3
- J4: renamed from J3; footprint Connector_JST:JST_XH_B3B-XH-A_1x03_P2.50mm_Vertical -> Connector_Molex:Molex_CLIK-Mate_502585-0370_1x03-1MP_P1.50mm_Horizontal
- J5: renamed from J4; footprint Connector_JST:JST_XH_B4B-XH-A_1x04_P2.50mm_Vertical -> Connector_Molex:Molex_CLIK-Mate_502585-0470_1x04-1MP_P1.50mm_Horizontal
- J7: renamed from J5; footprint Connector_JST:JST_XH_B4B-XH-A_1x04_P2.50mm_Vertical -> Connector_Molex:Molex_CLIK-Mate_502585-0470_1x04-1MP_P1.50mm_Horizontal
- J8: renamed from J6; footprint Connector_JST:JST_XH_B4B-XH-A_1x04_P2.50mm_Vertical -> Connector_Molex:Molex_CLIK-Mate_502585-0470_1x04-1MP_P1.50mm_Horizontal
- J9: renamed from J7; footprint Connector_JST:JST_XH_B4B-XH-A_1x04_P2.50mm_Vertical -> Connector_Molex:Molex_CLIK-Mate_502585-0470_1x04-1MP_P1.50mm_Horizontal
- R17: renamed from R12; value 220 -> 10K
- moved H1 225.8 mm to (-46.3, 111.3)
- moved H2 225.8 mm to (-46.3, 61.3)
- moved H3 225.8 mm to (-96.3, 111.3)
- moved H4 225.8 mm to (-96.3, 61.3)
- moved C13 104.8 mm to (269.2, 128.8)
- moved C14 104.8 mm to (266.5, 131.2)
- moved C16 104.8 mm to (266.5, 132.8)
- moved C19 104.8 mm to (262.0, 125.8)
- moved L2 104.8 mm to (274.5, 128.8)
- moved C11 104.8 mm to (277.1, 129.6)
- moved C12 104.8 mm to (271.8, 129.6)
- moved C15 104.8 mm to (267.6, 124.3)
- moved C17 104.8 mm to (267.6, 125.8)
- moved IC1 104.8 mm to (263.0, 128.8)
- moved J2 104.8 mm to (280.7, 128.9)
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- renumbered C8 to C10, C9 to C11, C10 to C12, C11 to C13, C12 to C14, C13 to C15, C14 to C16, C15 to C17, C21 to C19, C16 to C21, C18 to C22, C19 to C23, C22 to C25, C28 to C27, C30 to C28, C2 to C3, C20 to C31, C24 to C32, C25 to C33, C27 to C34, C37 to C35, C38 to C36, C40 to C37, C41 to C38, C3 to C4, C4 to C5, C5 to C6, C6 to C8, C7 to C9, D3 to D4, Q1 to Q4, Q2 to Q5, Q3 to Q7, Q4 to Q8, R6 to R11, R7 to R12, R8 to R13, R9 to R14, R10 to R15, R11 to R16, R1 to R2, R13 to R21, R14 to R22, R15 to R23, R16 to R25, R17 to R26, R2 to R3, R3 to R4, R4 to R6, R5 to R9, U2 to U3, U3 to U4
Connections:
- net /AirLora V3/MCU/PA11 renamed /AirLora V3/MCU Sub/PA1
- net VREF+ renamed Net-(U5-VDDA)
- C10 pad 1: VDDRF -> +3.3V
- C14 pad 1: Net-(U3-VDD) -> GND
- C14 pad 2: GND -> Net-(U4-VDD)
- C16 pad 1: Net-(U3-VDD) -> GND
- C16 pad 2: GND -> Net-(U4-VDD)
- C23 pad 1: VDDPA -> VDDRF1V55
- C24 pad 1: Net-(C34-Pad1) -> Net-(U5-OSC_OUT)
- C24 pad 2: XTA -> GND
- C26 pad 1: VDDRF -> +3.3V
- C31 pad 1: VDDRF -> +3.3V
- C32 pad 1: VDDRF -> +3.3V
- C33 pad 1: VDDRF -> +3.3V
- C34 pad 1: VDDRF -> +3.3V
- C37 pad 1: VDDPA -> VDDRF1V55
- C39 pad 1: VDDPA -> 3.3V
- D4 pad 2: VDDRF -> +3.3V
- J1 pad 1: Net-(D1-A) -> Net-(J1-Pin_1)
- J5 pad 3: /AirLora V3/MCU/PA9_TX -> /AirLora V3/MCU Sub/RX3
- J5 pad 4: /AirLora V3/MCU/PA10_RX -> /AirLora V3/MCU Sub/TX3
- J7 pad 3: /AirLora V3/MCU/PA3_RX -> /AirLora V3/MCU Sub/TX2
- J7 pad 4: /AirLora V3/MCU/PA2_TX -> /AirLora V3/MCU Sub/RX2
- J8 pad 3: /AirLora V3/MCU/PB8_SCL -> /AirLora V3/MCU Sub/SDA1
- J8 pad 4: /AirLora V3/MCU/PB9_SDA -> /AirLora V3/MCU Sub/SCL1
- J9 pad 2: VDDRF -> +3.3V
- J9 pad 3: /AirLora V3/MCU/T_SWCLK -> Net-(J9-Pin_3)
- J9 pad 4: /AirLora V3/MCU/T_SWDIO -> Net-(J9-Pin_4)
- L3 pad 1: VDDPA -> VDDRF1V55
- L4 pad 1: VDDRF -> +3.3V
- R11 pad 2: VDDRF -> +3.3V
- R12 pad 1: VDDRF -> +3.3V
- R15 pad 1: VDDRF -> +3.3V
- R15 pad 2: Net-(U3-VDD) -> Net-(U4-VDD)
- R17 pad 1: Net-(XTAL1-OUTPUT) -> GND
- R17 pad 2: Net-(C34-Pad1) -> Net-(U5-PH3)
- R2 pad 2: /AirLora V3/MCU/PA12 -> /AirLora V3/MCU/PB3
- R22 pad 2: /AirLora V3/MCU/PB2 -> /AirLora V3/MCU Sub/PA7
- R23 pad 1: /AirLora V3/MCU/PA6 -> /AirLora V3/MCU Sub/PA5
- R25 pad 1: /AirLora V3/MCU/PA5 -> /AirLora V3/MCU Sub/PA4
- R26 pad 1: /AirLora V3/MCU/PA8 -> /AirLora V3/MCU Sub/PA6
- U3 pad 1: VDDRF -> +3.3V
- U4 pad 4: Net-(U3-VDD) -> Net-(U4-VDD)
Routing:
- net +5V: track 140.1 -> 24.1 mm, vias 4 -> 0
- net VDDRF: track 79.7 -> 15.0 mm, vias 13 -> 0
- net /AirLora V3/MCU/PA12: track 42.7 -> 0.00 mm, vias 2 -> 0
- net /AirLora V3/MCU/PB9_SDA: track 37.8 -> 0.00 mm, vias 1 -> 0
- net 12V: track 37.1 -> 0.00 mm
- net +3.3V: track 0.00 -> 33.1 mm, vias 0 -> 5
- net /AirLora V3/MCU/PA9_TX: track 32.7 -> 0.00 mm, vias 1 -> 0
- net /AirLora V3/MCU/PB8_SCL: track 31.4 -> 0.00 mm, vias 1 -> 0
- net /AirLora V3/MCU/T_SWDIO: track 27.4 -> 0.00 mm, vias 1 -> 0
- net /AirLora V3/MCU/T_SWCLK: track 27.2 -> 1.76 mm
- net /AirLora V3/MCU Sub/PA1: track 33.6 -> 8.47 mm, vias 1 -> 0
- net /AirLora V3/MCU/PA5: track 25.1 -> 0.00 mm, vias 2 -> 0
- net /AirLora V3/MCU/PB2: track 24.7 -> 0.00 mm, vias 3 -> 0
- net /AirLora V3/MCU/PA10_RX: track 24.2 -> 0.00 mm, vias 1 -> 0
- net /AirLora V3/MCU/PA2_TX: track 23.2 -> 0.00 mm, vias 1 -> 0
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- removed copper zone on In2.Cu, net VDDPA
