File: PCBDesign/AirLoRaV3_PCBDesign/airlora_v3.kicad_sch (KiCad schematic)
At the start: 0 parts

Commit message: Update PCB
Other:
- sheet MCU ports: added PA3; removed PB3
Changed lines of the file:
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@@
+	(wire
+		(pts
+			(xy 167.64 105.41) (xy 190.5 105.41)
+		)
+		(stroke
+			(width 0)
+			(type default)
+		)
+	)
 	(wire
 		(pts
@@
 	(wire
 		(pts
+			(xy 165.1 63.5) (xy 179.07 63.5)
+		)
+		(stroke
+			(width 0)
+			(type default)
+		)
+	)
+	(wire
+		(pts
+			(xy 167.64 142.24) (xy 190.5 142.24)
+		)
+		(stroke
+			(width 0)
+			(type default)
+		)
+	)
+	(wire
+		(pts
+			(xy 185.42 125.73) (xy 185.42 116.84)
+		)
+		(stroke
+			(width 0)
+			(type default)
+		)
+	)
+	(wire
+		(pts
+			(xy 185.42 134.62) (xy 185.42 125.73)
+		)
+		(stroke
+			(width 0)
+			(type default)
+		)
+	)
+	(wire
+		(pts
+			(xy 96.52 107.95) (xy 107.95 107.95)
+		)
+		(stroke
+			(width 0)
+			(type default)
+		)
+	)
+	(wire
+		(pts
+			(xy 175.26 90.17) (xy 175.26 66.04)
+		)
+		(stroke
+			(width 0)
+			(type default)
+		)
+	)
+	(wire
+		(pts
 			(xy 167.64 114.3) (xy 190.5 114.3)
 		)
@@
 	(wire
 		(pts
-			(xy 165.1 63.5) (xy 179.07 63.5)
-		)
-		(stroke
-			(width 0)
-			(type default)
-		)
-	)
-	(wire
-		(pts
-			(xy 167.64 142.24) (xy 190.5 142.24)
-		)
-		(stroke
-			(width 0)
-			(type default)
-		)
-	)
-	(wire
-		(pts
-			(xy 185.42 125.73) (xy 185.42 116.84)
-		)
-		(stroke
-			(width 0)
-			(type default)
-		)
-	)
-	(wire
-		(pts
-			(xy 185.42 134.62) (xy 185.42 125.73)
-		)
-		(stroke
-			(width 0)
-			(type default)
-		)
-	)
-	(wire
-		(pts
-			(xy 96.52 107.95) (xy 107.95 107.95)
-		)
-		(stroke
-			(width 0)
-			(type default)
-		)
-	)
-	(wire
-		(pts
-			(xy 175.26 90.17) (xy 175.26 66.04)
-		)
-		(stroke
-			(width 0)
-			(type default)
-		)
-	)
-	(wire
-		(pts
 			(xy 132.08 54.61) (xy 107.95 54.61)
 		)
@@
 		(pts
 			(xy 167.64 87.63) (xy 179.07 87.63)
-		)
-		(stroke
-			(width 0)
-			(type default)
-		)
-	)
-	(wire
-		(pts
-			(xy 167.64 105.41) (xy 190.5 105.41)
 		)
 		(stroke
@@
 			)
 		)
-		(pin "PB3" input
+		(pin "PA3" input
 			(at 132.08 67.31 180)
 			(effects
@@
 		)
 		(pin "PA6" input
-			(at 167.64 105.41 0)
+			(at 167.64 149.86 0)
 			(effects
 				(font
@@
 		)
 		(pin "PA4" input
-			(at 167.64 114.3 0)
+			(at 167.64 142.24 0)
 			(effects
 				(font
@@
 		)
 		(pin "PB3" input
-			(at 167.64 142.24 0)
+			(at 167.64 114.3 0)
 			(effects
 				(font
@@
 		)
 		(pin "PB4" input
-			(at 167.64 149.86 0)
-			(effects
-				(font
+			(at 167.64 105.41 0)
+			(effects
+				(font
