File: PCBDesign/AirLoRaV3_PCBDesign/MCU.kicad_sch (KiCad schematic)
At the start: 50 parts, among them IC1 BALFHB-WL-02D3, J2 Conn_Coaxial, J3 Led, Q2 S8050, Q3 S8050, SW1 SW_Push, U4 BGS12WN6E6327, U5 STM32WLE5CCUx, X1 NX2016SA-32MHZ, Y1 NX2012SA 32.768KHz

Commit message: Update package and placement components
Parts:
- added C47: 0.47uF, Capacitor_SMD:C_0402_1005Metric_Pad0.74x0.62mm_HandSolder, symbol Device:C
- added C48: 470nF, Capacitor_SMD:C_0402_1005Metric_Pad0.74x0.62mm_HandSolder, symbol Device:C
- added C49, C50: 100pF, Capacitor_SMD:C_0402_1005Metric_Pad0.74x0.62mm_HandSolder, symbol Device:C
- added L5: NC, Inductor_SMD:L_0402_1005Metric_Pad0.77x0.64mm_HandSolder, symbol Device:L
- C11, C12, C13, C14, C15, C16, C17, C18, C19, C20, C21, C22, C23, C24, C25, C26, C27, C28, C29, C30, C31, C32, C33, C34, C36, C37: footprint Capacitor_SMD:C_0603_1608Metric -> Capacitor_SMD:C_0402_1005Metric_Pad0.74x0.62mm_HandSolder
- C35: value 33pF -> 100pF; footprint Capacitor_SMD:C_0603_1608Metric -> Capacitor_SMD:C_0402_1005Metric_Pad0.74x0.62mm_HandSolder
- L2, L4: footprint Inductor_SMD:L_0603_1608Metric -> Inductor_SMD:L_0402_1005Metric_Pad0.77x0.64mm_HandSolder
- L3: footprint Capacitor_SMD:C_0603_1608Metric_Pad1.08x0.95mm_HandSolder -> Inductor_SMD:L_0402_1005Metric_Pad0.77x0.64mm_HandSolder
- R15, R16, R17, R18, R19, R20: footprint Resistor_SMD:R_0603_1608Metric -> Resistor_SMD:R_0402_1005Metric_Pad0.72x0.64mm_HandSolder
Connections:
- net GND: now also C47.2, C48.2, C49.2, C50.2
- net VDDPA: now also C50.1
- net VDDRF: now also C49.1
- net RFO_IN: now reaches C19.2, U5.23 (RFO_HP)
- net RFO_IN: now also L5.2
- net at U5.24 (VR_PA): now also C47.1, C48.1, L5.1
- no-connect marks 20 -> 19
Other:
- moved on the sheet: C19, C31, C32, C33, C34, C35, C36, C37
