File: airlora_v3.kicad_sch (KiCad schematic)
At the start: 0 parts

Commit message: Update schematic
Connections:
- no-connect marks 3 -> 0
Other:
- removed sheet MCU Sub
- sheet MCU ports: added NRST, PA5, PB12, PB2, PB7, SCL3, SDA3, UART2_RX, UART2_TX; removed PA3, PA4
- sheet STlink ports: added NRST; removed T_SWCLK1, T_SWDIO1
