File: MCU.kicad_sch (KiCad schematic)
At the start: 56 parts, among them IC1 BALFHB-WL-02D3, J12 UART_MAIN, J2 Conn_Coaxial, J3 Led, Q1 S8050, Q2 S8050, SW1 SW_Push, U4 BGS12WN6E6327, U5 STM32WLE5CCUx, X1 32MHZ, Y1 32.768kHz

Commit message: Update schematic
Parts:
- removed J12: UART_MAIN, Connector_JST:JST_XH_B4B-XH-A_1x04_P2.50mm_Vertical, symbol Connector:Screw_Terminal_01x04
- removed R16: 1K, Resistor_SMD:R_0402_1005Metric, symbol Device:R
- removed X1: 32MHZ, footprint:NX2016SA_NDK, symbol NX2016SA-32MHZ:NX2016SA-32MHZ-EXS00A-CS06654
- added J13: UART_MAIN, Connector_JST:JST_XH_B3B-XH-A_1x03_P2.50mm_Vertical, symbol Connector:Screw_Terminal_01x03
- added L6: 1400R@1GHz, Inductor_SMD:L_0402_1005Metric, symbol Device:L
- added R10: 220, Resistor_SMD:R_0402_1005Metric, symbol Device:R
- added TP1, TP2, TP3, TP4, TP5, TP6: TestPoint, symbol Connector:TestPoint
- added XTAL1: NT2016SA-32M-END4263A, footprint:NT2016SA-32M-END4263A_NDK, symbol NT2016SA-32M-:NT2016SA-32M-END4263A
- C37, C41: value 6.8pF -> 10pF
Connections:
- net GND: now also C37.2, J13.3 (Pin_3), XTAL1.1 (GND), XTAL1.2 (GND); no longer C37.1, C41.2
- net PA5: no longer R18.1
- net SCL2: now also U5.35 (PA12), TP5.1; no longer U5.34 (PA11)
- net SDA2: now also U5.34 (PA11), TP6.1; no longer U5.35 (PA12)
- net UART1_RX: now also U5.33 (PA10), J13.1 (Pin_1); no longer U5.5 (PB7)
- net UART1_TX: now also U5.17 (PA9), J13.2 (Pin_2); no longer U5.4 (PB6)
- net SCL3: now reaches U5.15 (PA7)
- net SCL3: now also TP3.1
- net SDA3: now reaches U5.2 (PB4)
- net SDA3: now also TP4.1
- net XTA: now reaches U5.26 (OSC_IN)
- net XTA: now also C41.1; no longer C37.2
- net at U5.27 (OSC_OUT): no longer C41.1
- net PB5: now reaches U5.3 (PB5)
- net PB5: now also R18.1
- net PB0: now reaches U5.30 (PB0-VDD_TCXO)
- net PB0: now also L6.1
- net PB2: now reaches U5.31 (PB2)
- net PB12: now reaches U5.32 (PB12)
- net UART2_TX: now reaches U5.9 (PA2)
- net UART2_TX: now also TP2.1
- net PA3 renamed UART2_RX
- net UART2_RX: now also TP1.1
- net PA6: no longer names the net of U5.14 (PA6)
- net PA6: no longer R19.1
- new net: R10.1, XTAL1.3 (OUTPUT)
- new net: C37.1, L6.2, XTAL1.4 (VCC)
- new net: C41.2, R10.2
- new net PB6: R19.1, U5.4 (PB6)
- new net PB7: U5.5 (PB7)
- no-connect marks 16 -> 10
Other:
- moved on the sheet: C34, C35, C37, C38, C39, C40, C41

Commit message: Udpate test point
Connections:
- net PA5: no longer names the net of U5.13 (PA5)
- net PB12: no longer names the net of U5.32 (PB12)
- net PB2: no longer names the net of U5.31 (PB2)
- no-connect marks 10 -> 11
Changed lines of the file:
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@@
+	)
+	(no_connect
+		(at 215.9 147.32)
 	)
 	(no_connect
@@
 	(wire
 		(pts
-			(xy 256.54 119.38) (xy 259.08 119.38)
-		)
-		(stroke
-			(width 0)
-			(type default)
-		)
-	)
-	(wire
-		(pts
 			(xy 257.81 109.22) (xy 259.08 109.22)
 		)
@@
 	(wire
 		(pts
-			(xy 256.54 116.84) (xy 259.08 116.84)
-		)
-		(stroke
-			(width 0)
-			(type default)
-		)
-	)
-	(wire
-		(pts
 			(xy 241.3 147.32) (xy 241.3 207.01)
 		)
@@
 		(pts
 			(xy 266.7 127) (xy 266.7 138.43)
-		)
-		(stroke
-			(width 0)
-			(type default)
-		)
-	)
-	(wire
-		(pts
-			(xy 215.9 147.32) (xy 215.9 151.13)
 		)
 		(stroke
@@
 		)
 	)
-	(hierarchical_label "PB12"
-		(shape input)
-		(at 259.08 116.84 0)
-		(fields_autoplaced yes)
-		(effects
-			(font
-				(size 1.27 1.27)
-			)
-			(justify left)
-		)
-	)
-	(hierarchical_label "PA5"
-		(shape input)
-		(at 215.9 151.13 270)
-		(fields_autoplaced yes)
-		(effects
-			(font
-				(size 1.27 1.27)
-			)
-			(justify right)
-		)
-	)
 	(hierarchical_label "SDA2"
 		(shape input)
@@
 		)
 	)
-	(hierarchical_label "PB2"
-		(shape input)
-		(at 259.08 119.38 0)
-		(fields_autoplaced yes)
-		(effects
-			(font
-				(size 1.27 1.27)
-			)
-			(justify left)
-		)
-	)
