File: STlink.kicad_sch (KiCad schematic)
At the start: 2 parts, among them J11 UART2, SW2 SW_Slide_DPDT

Commit message: Update schematic
Parts:
- removed J11: UART2, Connector_JST:JST_XH_B4B-XH-A_1x04_P2.50mm_Vertical, symbol Connector:Screw_Terminal_01x04
- removed SW2: SW_Slide_DPDT, Button_Switch_THT:SW_E-Switch_EG1271_SPDT, symbol Switch:SW_Slide_DPDT
- added J12: STlink, symbol Connector:Screw_Terminal_01x05
Connections:
- net +3.3V: now also J12.1 (Pin_1)
- net GND: now also J12.2 (Pin_2)
- net T_SWCLK: now also J12.4 (Pin_4)
- net T_SWDIO: now also J12.3 (Pin_3)
- new net NRST: J12.5 (Pin_5)

Commit message: Update PCB layout
Parts:
- J12: footprint (none) -> Connector_JST:JST_XH_B5B-XH-A_1x05_P2.50mm_Vertical
Changed lines of the file:
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@@
 			)
 		)
-		(property "Footprint" ""
+		(property "Footprint" "Connector_JST:JST_XH_B5B-XH-A_1x05_P2.50mm_Vertical"
 			(at 156.21 88.9 0)
 			(effects
